File: esp32.kicad_sch (KiCad schematic)
At the start: 13 parts, among them IC3 ESP32-C3-WROOM-02-N4, J5 UART, J6 ToSSR, Q1 BSS138, SW1 SW_Push

Commit message: fix: J5 and J6 FP to 2.54mm headers
Parts:
- J5: footprint Connector_PinHeader_1.00mm:PinHeader_1x04_P1.00mm_Vertical -> Connector_PinHeader_2.54mm:PinHeader_1x04_P2.54mm_Vertical
- J6: footprint Connector_PinHeader_1.00mm:PinHeader_1x01_P1.00mm_Horizontal -> Connector_PinHeader_2.54mm:PinHeader_1x01_P2.54mm_Vertical
Changed lines of the file:
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@@
       (effects (font (size 1.27 1.27)))
     )
-    (property "Footprint" "Connector_PinHeader_1.00mm:PinHeader_1x04_P1.00mm_Vertical" (at 27.94 144.78 0)
+    (property "Footprint" "Connector_PinHeader_2.54mm:PinHeader_1x04_P2.54mm_Vertical" (at 27.94 144.78 0)
       (effects (font (size 1.27 1.27)) hide)
     )
@@
       (effects (font (size 1.27 1.27)))
     )
-    (property "Footprint" "Connector_PinHeader_1.00mm:PinHeader_1x01_P1.00mm_Horizontal" (at 152.4 55.88 0)
+    (property "Footprint" "Connector_PinHeader_2.54mm:PinHeader_1x01_P2.54mm_Vertical" (at 152.4 55.88 0)
       (effects (font (size 1.27 1.27)) hide)
     )
