File: power.kicad_sch (KiCad schematic)
At the start: 8 parts, among them IC2 L6981C33DR, J3 Barrel_Jack_Switch_Pin3Ring

Commit message: fix: init symbols references
Parts:
- renumbered D2 to D1, IC2 to IC1, J3 to J1
Changed lines of the file:
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@@
   (symbol (lib_id "Connector:Barrel_Jack_Switch_Pin3Ring") (at 71.12 71.12 0) (unit 1)
     (in_bom yes) (on_board yes) (dnp no) (fields_autoplaced)
-    (property "Reference" "J3" (at 71.12 62.23 0)
+    (property "Reference" "J1" (at 71.12 62.23 0)
       (effects (font (size 1.27 1.27)))
     )
@@
       (project "pv_router"
         (path "/08ef31dc-81c2-4bcd-8336-e62c344e451e/760387e1-ffe6-428e-8651-2617e5a76fa2"
-          (reference "J3") (unit 1)
+          (reference "J1") (unit 1)
         )
       )
@@
   (symbol (lib_id "power:GND") (at 86.36 73.66 0) (unit 1)
     (in_bom yes) (on_board yes) (dnp no) (fields_autoplaced)
-    (property "Reference" "#PWR06" (at 86.36 80.01 0)
+    (property "Reference" "#PWR01" (at 86.36 80.01 0)
       (effects (font (size 1.27 1.27)) hide)
     )
@@
       (project "pv_router"
         (path "/08ef31dc-81c2-4bcd-8336-e62c344e451e/760387e1-ffe6-428e-8651-2617e5a76fa2"
-          (reference "#PWR06") (unit 1)
+          (reference "#PWR01") (unit 1)
         )
       )
@@
   (symbol (lib_id "power:GND") (at 154.94 96.52 0) (unit 1)
     (in_bom yes) (on_board yes) (dnp no) (fields_autoplaced)
-    (property "Reference" "#PWR08" (at 154.94 102.87 0)
+    (property "Reference" "#PWR03" (at 154.94 102.87 0)
       (effects (font (size 1.27 1.27)) hide)
     )
@@
       (project "pv_router"
         (path "/08ef31dc-81c2-4bcd-8336-e62c344e451e/760387e1-ffe6-428e-8651-2617e5a76fa2"
-          (reference "#PWR08") (unit 1)
+          (reference "#PWR03") (unit 1)
         )
       )
@@
   (symbol (lib_id "L6981C33DR:L6981C33DR") (at 172.72 60.96 0) (mirror y) (unit 1)
     (in_bom yes) (on_board yes) (dnp no)
-    (property "Reference" "IC2" (at 153.67 53.34 0)
+    (property "Reference" "IC1" (at 153.67 53.34 0)
       (effects (font (size 1.27 1.27)))
     )
@@
       (project "pv_router"
         (path "/08ef31dc-81c2-4bcd-8336-e62c344e451e/760387e1-ffe6-428e-8651-2617e5a76fa2"
-          (reference "IC2") (unit 1)
+          (reference "IC1") (unit 1)
         )
       )
@@
   (symbol (lib_id "Diode:PMEG6020ELR") (at 97.79 68.58 180) (unit 1)
     (in_bom yes) (on_board yes) (dnp no) (fields_autoplaced)
-    (property "Reference" "D2" (at 98.1075 62.23 0)
+    (property "Reference" "D1" (at 98.1075 62.23 0)
       (effects (font (size 1.27 1.27)))
     )
@@
       (project "pv_router"
         (path "/08ef31dc-81c2-4bcd-8336-e62c344e451e/760387e1-ffe6-428e-8651-2617e5a76fa2"
-          (reference "D2") (unit 1)
+          (reference "D1") (unit 1)
         )
       )
@@
   (symbol (lib_id "power:GND") (at 119.38 40.64 0) (unit 1)
     (in_bom yes) (on_board yes) (dnp no) (fields_autoplaced)
-    (property "Reference" "#PWR026" (at 119.38 46.99 0)
+    (property "Reference" "#PWR02" (at 119.38 46.99 0)
       (effects (font (size 1.27 1.27)) hide)
     )
@@
       (project "pv_router"
         (path "/08ef31dc-81c2-4bcd-8336-e62c344e451e/760387e1-ffe6-428e-8651-2617e5a76fa2"
-          (reference "#PWR026") (unit 1)
+          (reference "#PWR02") (unit 1)
         )
       )
@@
   (symbol (lib_id "power:+3V3") (at 243.84 60.96 0) (unit 1)
     (in_bom yes) (on_board yes) (dnp no) (fields_autoplaced)
-    (property "Reference" "#PWR05" (at 243.84 64.77 0)
+    (property "Reference" "#PWR04" (at 243.84 64.77 0)
       (effects (font (size 1.27 1.27)) hide)
     )
@@
       (project "pv_router"
         (path "/08ef31dc-81c2-4bcd-8336-e62c344e451e/760387e1-ffe6-428e-8651-2617e5a76fa2"
+          (reference "#PWR04") (unit 1)
+        )
+      )
+    )
+  )
+  (symbol (lib_id "power:+3V3") (at 246.38 38.1 0) (unit 1)
+    (in_bom yes) (on_board yes) (dnp no) (fields_autoplaced)
+    (property "Reference" "#PWR05" (at 246.38 41.91 0)
+      (effects (font (size 1.27 1.27)) hide)
+    )
+    (property "Value" "+3V3" (at 246.38 33.02 0)
+      (effects (font (size 1.27 1.27)))
+    )
+    (property "Footprint" "" (at 246.38 38.1 0)
+      (effects (font (size 1.27 1.27)) hide)
+    )
+    (property "Datasheet" "" (at 246.38 38.1 0)
+      (effects (font (size 1.27 1.27)) hide)
+    )
+    (pin "1")
+    (instances
+      (project "pv_router"
+        (path "/08ef31dc-81c2-4bcd-8336-e62c344e451e/760387e1-ffe6-428e-8651-2617e5a76fa2"
           (reference "#PWR05") (unit 1)
         )
       )
-    )
-  )
-  (symbol (lib_id "power:+3V3") (at 246.38 38.1 0) (unit 1)
-    (in_bom yes) (on_board yes) (dnp no) (fields_autoplaced)
-    (property "Reference" "#PWR027" (at 246.38 41.91 0)
-      (effects (font (size 1.27 1.27)) hide)
-    )
-    (property "Value" "+3V3" (at 246.38 33.02 0)
-      (effects (font (size 1.27 1.27)))
-    )
-    (property "Footprint" "" (at 246.38 38.1 0)
-      (effects (font (size 1.27 1.27)) hide)
-    )
-    (property "Datasheet" "" (at 246.38 38.1 0)
-      (effects (font (size 1.27 1.27)) hide)
-    )
-    (pin "1")
-    (instances
-      (project "pv_router"
-        (path "/08ef31dc-81c2-4bcd-8336-e62c344e451e/760387e1-ffe6-428e-8651-2617e5a76fa2"
-          (reference "#PWR027") (unit 1)
-        )
-      )

Commit message: fix: assigned FP for ICs
Parts:
- IC1: footprint SOIC127P600X175-8N -> L6981C33DR:SOIC127P600X175-8N
Changed lines of the file:
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@@
       (effects (font (size 1.27 1.27)))
     )
-    (property "Footprint" "SOIC127P600X175-8N" (at 138.43 155.88 0)
+    (property "Footprint" "L6981C33DR:SOIC127P600X175-8N" (at 138.43 155.88 0)
       (effects (font (size 1.27 1.27)) (justify left top) hide)
     )

Commit message: pcb: fix inductor value to 33uH
Parts:
- L1: value 3.3uH -> 33uH; footprint Inductor_SMD:L_10.4x10.4_H4.8 -> MSS1038T-333MLC:MSS1038T333MLC
Changed lines of the file:
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@@
       (effects (font (size 1.27 1.27)))
     )
-    (property "Value" "3.3uH" (at 226.06 58.42 90)
+    (property "Value" "33uH" (at 226.06 58.42 90)
       (effects (font (size 1.27 1.27)))
     )
-    (property "Footprint" "Inductor_SMD:L_10.4x10.4_H4.8" (at 226.06 60.96 0)
+    (property "Footprint" "MSS1038T-333MLC:MSS1038T333MLC" (at 226.06 60.96 0)
       (effects (font (size 1.27 1.27)) hide)
     )

Commit message: FP: first FP update
Parts:
- Cvcc1: footprint Capacitor_SMD:C_0805_2012Metric_Pad1.18x1.45mm_HandSolder -> Capacitor_SMD:C_0603_1608Metric
Changed lines of the file:
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@@
       (effects (font (size 1.27 1.27)) (justify left))
     )
-    (property "Footprint" "Capacitor_SMD:C_0805_2012Metric_Pad1.18x1.45mm_HandSolder" (at 191.4652 86.36 0)
+    (property "Footprint" "Capacitor_SMD:C_0603_1608Metric" (at 191.4652 86.36 0)
       (effects (font (size 1.27 1.27)) hide)
     )
-    (property "Datasheet" "~" (at 190.5 82.55 0)
+    (property "Datasheet" "1 dispo" (at 190.5 82.55 0)
       (effects (font (size 1.27 1.27)) hide)
     )

Commit message: FP: associate FP except jumpers
Parts:
- Cboot1, Cin1, Cout1: footprint Capacitor_SMD:C_0805_2012Metric_Pad1.18x1.45mm_HandSolder -> Capacitor_SMD:C_0805_2012Metric
- J1: footprint Connector_BarrelJack:BarrelJack_Wuerth_6941xx301002 -> Connector_BarrelJack:BarrelJack_CUI_PJ-079BH_Horizontal
Changed lines of the file:
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@@
       (effects (font (size 1.27 1.27)))
     )
-    (property "Footprint" "Connector_BarrelJack:BarrelJack_Wuerth_6941xx301002" (at 72.39 72.136 0)
-      (effects (font (size 1.27 1.27)) hide)
-    )
-    (property "Datasheet" "~" (at 72.39 72.136 0)
+    (property "Footprint" "Connector_BarrelJack:BarrelJack_CUI_PJ-079BH_Horizontal" (at 72.39 72.136 0)
+      (effects (font (size 1.27 1.27)) hide)
+    )
+    (property "Datasheet" "ok 2 !!FP" (at 72.39 72.136 0)
       (effects (font (size 1.27 1.27)) hide)
     )
@@
       (effects (font (size 1.27 1.27)) (justify left))
     )
-    (property "Footprint" "Capacitor_SMD:C_0805_2012Metric_Pad1.18x1.45mm_HandSolder" (at 211.7852 86.36 0)
+    (property "Footprint" "Capacitor_SMD:C_0805_2012Metric" (at 211.7852 86.36 0)
       (effects (font (size 1.27 1.27)) hide)
     )
@@
       (effects (font (size 1.27 1.27)) (justify right))
     )
-    (property "Footprint" "Capacitor_SMD:C_0805_2012Metric_Pad1.18x1.45mm_HandSolder" (at 131.1148 78.74 0)
+    (property "Footprint" "Capacitor_SMD:C_0805_2012Metric" (at 131.1148 78.74 0)
       (effects (font (size 1.27 1.27)) hide)
     )
@@
       (effects (font (size 1.27 1.27)))
     )
-    (property "Footprint" "Capacitor_SMD:C_0805_2012Metric_Pad1.18x1.45mm_HandSolder" (at 210.82 62.5348 0)
-      (effects (font (size 1.27 1.27)) hide)
-    )
-    (property "Datasheet" "~" (at 207.01 63.5 0)
-      (effects (font (size 1.27 1.27)) hide)
-    )
+    (property "Footprint" "Capacitor_SMD:C_0805_2012Metric" (at 210.82 62.5348 0)
+      (effects (font (size 1.27 1.27)) hide)
+    )
+    (property "Datasheet" "ok: 1" (at 207.01 63.5 0)
+      (effects (font (size 1.27 1.27)) hide)
+    )

Commit message: fix: delete diode on input supply ic
Parts:
- removed D1: PMEG6020ELR, Diode_SMD:Nexperia_CFP3_SOD-123W, symbol Diode:PMEG6020ELR
Connections:
- net at J1.1: now also Cin1.2, IC1.5 (EN/CLKIN), IC1.7 (VIN)
Changed lines of the file:
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@@
-    (stroke (width 0) (type default))
-  )
-  (wire (pts (xy 78.74 68.58) (xy 93.98 68.58))
     (stroke (width 0) (type default))
   )
@@
     (stroke (width 0) (type default))
   )
-  (wire (pts (xy 101.6 68.58) (xy 132.08 68.58))
+  (wire (pts (xy 78.74 68.58) (xy 132.08 68.58))
     (stroke (width 0) (type default))
   )
@@
         )
       )
-    )
-  )
-  (symbol (lib_id "Diode:PMEG6020ELR") (at 97.79 68.58 180) (unit 1)
-    (in_bom yes) (on_board yes) (dnp no) (fields_autoplaced)
-    (property "Reference" "D1" (at 98.1075 62.23 0)
-      (effects (font (size 1.27 1.27)))
-    )
-    (property "Value" "PMEG6020ELR" (at 98.1075 64.77 0)
-      (effects (font (size 1.27 1.27)))
-    )
-    (property "Footprint" "Diode_SMD:Nexperia_CFP3_SOD-123W" (at 97.79 64.135 0)
-      (effects (font (size 1.27 1.27)) hide)
-    )
-    (property "Datasheet" "https://assets.nexperia.com/documents/data-sheet/PMEG6020ELR.pdf" (at 97.79 68.58 0)
-      (effects (font (size 1.27 1.27)) hide)
-    )
-    (pin "2")
-    (pin "1")
-    (instances
-      (project "pv_router"
-        (path "/08ef31dc-81c2-4bcd-8336-e62c344e451e/760387e1-ffe6-428e-8651-2617e5a76fa2"
-          (reference "D1") (unit 1)
-        )
-      )

Commit message: fix: barrel jack FP on PCB
Parts:
- J1: footprint Connector_BarrelJack:BarrelJack_CUI_PJ-079BH_Horizontal -> BarrelJack:BarrelJack_CUI_PJ-051A_Horizontal
Changed lines of the file:
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@@
       (effects (font (size 1.27 1.27)))
     )
-    (property "Footprint" "Connector_BarrelJack:BarrelJack_CUI_PJ-079BH_Horizontal" (at 72.39 72.136 0)
+    (property "Footprint" "BarrelJack:BarrelJack_CUI_PJ-051A_Horizontal" (at 72.39 72.136 0)
       (effects (font (size 1.27 1.27)) hide)
     )
