File: adc.kicad_sch (KiCad schematic)
At the start: 33 parts, among them IC2 ATM90E26-YU-B, J2 AudioJack3, J3 AudioJack3, J4 Barrel_Jack_Switch_Pin3Ring, Y1 8.192Mhz

Commit message: fix: after ERC check
Parts:
- IC2: footprint ATM90E26-YU-B:SOP65P778X199-28N -> SOP65P778X199-28N
Changed lines of the file:
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@@
 			)
 		)
-		(property "Datasheet" "ok : 4"
+		(property "Datasheet" "~"
 			(at 134.62 83.82 0)
 			(effects
@@
 			)
 		)
-		(property "Description" ""
+		(property "Description" "Unpolarized capacitor"
 			(at 134.62 83.82 0)
 			(effects
@@
 			)
 		)
-		(property "Datasheet" "ok : 6"
+		(property "Datasheet" "~"
 			(at 40.64 107.95 0)
 			(effects
@@
 			)
 		)
-		(property "Description" ""
+		(property "Description" "Resistor"
 			(at 40.64 107.95 0)
 			(effects
@@
 			)
 		)
-		(property "Description" ""
+		(property "Description" "Power symbol creates a global label with name \"GND\" , ground"
 			(at 55.88 114.3 0)
 			(effects
@@
 			)
 		)
-		(property "Description" ""
+		(property "Description" "Jumper, 2-pole, closed/bridged"
 			(at 167.64 45.72 0)
 			(effects
@@
 			)
 		)
-		(property "Description" ""
+		(property "Description" "Power symbol creates a global label with name \"GND\" , ground"
 			(at 76.2 154.94 0)
 			(effects
@@
 			)
 		)
-		(property "Datasheet" "ok : 6"
+		(property "Datasheet" "~"
 			(at 193.04 119.38 0)
 			(effects
@@
 			)
 		)
-		(property "Description" ""
+		(property "Description" "Unpolarized capacitor"
 			(at 193.04 119.38 0)
 			(effects
@@
 			)
 		)
-		(property "Description" ""
+		(property "Description" "Power symbol creates a global label with name \"GND\" , ground"
 			(at 121.92 114.3 0)
 			(effects
@@
 			)
 		)
-		(property "Description" ""
+		(property "Description" "Power symbol creates a global label with name \"+3V3\""
 			(at 172.72 40.64 0)
 			(effects
@@
 			)
 		)
-		(property "Datasheet" "ok : 6"
+		(property "Datasheet" "~"
 			(at 60.96 73.66 0)
 			(effects
@@
 			)
 		)
-		(property "Description" ""
+		(property "Description" "Unpolarized capacitor"
 			(at 60.96 73.66 0)
 			(effects
@@
 			)
 		)
-		(property "Description" ""
+		(property "Description" "Power symbol creates a global label with name \"GND\" , ground"
 			(at 223.52 127 0)
 			(effects
@@
 			)
 		)
-		(property "Description" ""
+		(property "Description" "Power symbol creates a global label with name \"GND\" , ground"
 			(at 121.92 63.5 0)
 			(effects
@@
 			)
 		)
-		(property "Description" ""
+		(property "Description" "Jumper, 2-pole, open"
 			(at 167.64 55.88 0)
 			(effects
@@
 			)
 		)
-		(property "Datasheet" "2 ok"
+		(property "Datasheet" "~"
 			(at 242.57 81.28 0)
 			(effects
@@
 			)
 		)
-		(property "Description" ""
+		(property "Description" "Unpolarized capacitor"
 			(at 242.57 81.28 0)
 			(effects
@@
 			)
 		)
-		(property "Description" ""
+		(property "Description" "Power symbol creates a global label with name \"GND\" , ground"
 			(at 172.72 60.96 0)
 			(effects
@@
 			)
 		)
-		(property "Datasheet" "ok : 6"
+		(property "Datasheet" "~"
 			(at 60.96 107.95 0)
 			(effects
@@
 			)
 		)
-		(property "Description" ""
+		(property "Description" "Unpolarized capacitor"
 			(at 60.96 107.95 0)
 			(effects
@@
 			)
 		)
-		(property "Datasheet" "ok 2 !!FP"
+		(property "Datasheet" "~"
 			(at 46.99 153.416 0)
 			(effects
@@
 			)
 		)
-		(property "Description" ""
+		(property "Description" "DC Barrel Jack with an internal switch"
 			(at 45.72 152.4 0)
 			(effects
@@
 			)
 		)
-		(property "Description" ""
+		(property "Description" "Jumper, 2-pole, open"
 			(at 177.8 55.88 0)
 			(effects
@@
 			)
 		)
-		(property "Description" ""
+		(property "Description" "Jumper, 2-pole, closed/bridged"
 			(at 177.8 45.72 0)
 			(effects
@@
 			)
 		)
-		(property "Footprint" "ATM90E26-YU-B:SOP65P778X199-28N"
+		(property "Footprint" "SOP65P778X199-28N"
 			(at 189.23 173.66 0)
 			(effects
@@
 			)
 		)
-		(property "Description" ""
+		(property "Description" "Atmel ATM90E26-YU-B Energy Measurement IC, 28-Pin SSOP"
 			(at 154.94 78.74 0)
 			(effects
@@
 			)
 		)
-		(property "Datasheet" "ok : 6"
+		(property "Datasheet" "~"
 			(at 40.64 83.82 0)
 			(effects
@@
 			)
 		)
-		(property "Description" ""
+		(property "Description" "Resistor"
 			(at 40.64 83.82 0)
 			(effects
@@
 			)
 		)
-		(property "Description" ""
+		(property "Description" "Power symbol creates a global label with name \"+3V3\""
 			(at 121.92 73.66 0)
 			(effects
@@
 			)
 		)
-		(property "Description" ""
+		(property "Description" "Power symbol creates a global label with name \"GND\" , ground"
 			(at 154.94 99.06 0)
 			(effects
@@
 			)
 		)
-		(property "Description" ""
+		(property "Description" "Power symbol creates a global label with name \"GND\" , ground"
 			(at 195.58 127 0)
 			(effects
@@
 			)
 		)
-		(property "Datasheet" "2 dispo en x7r 547-113-17"
+		(property "Datasheet" "~"
 			(at 134.62 116.84 0)
 			(effects
@@
 			)
 		)
-		(property "Description" ""
+		(property "Description" "Unpolarized capacitor"
 			(at 134.62 116.84 0)
 			(effects
@@
 			)
 		)
-		(property "Datasheet" "ok : 4"
+		(property "Datasheet" "~"
 			(at 142.24 67.31 0)
 			(effects
@@
 			)
 		)
-		(property "Description" ""
+		(property "Description" "Unpolarized capacitor"
 			(at 142.24 67.31 0)
 			(effects
@@
 			)
 		)
-		(property "Datasheet" "ok : 6"
+		(property "Datasheet" "~"
 			(at 40.64 72.39 0)
 			(effects
@@
 			)
 		)
-		(property "Description" ""
+		(property "Description" "Resistor"
 			(at 40.64 72.39 0)
 			(effects
@@
 			)
 		)
-		(property "Description" ""
+		(property "Description" "Power symbol creates a global label with name \"GND\" , ground"
 			(at 248.92 93.98 0)
 			(effects
@@
 			)
 		)
-		(property "Datasheet" "ok : 6"
+		(property "Datasheet" "~"
 			(at 233.68 118.11 0)
 			(effects
@@
 			)
 		)
-		(property "Description" ""
+		(property "Description" "Unpolarized capacitor"
 			(at 233.68 118.11 0)
 			(effects
@@
 			)
 		)
-		(property "Datasheet" "ok 2"
+		(property "Datasheet" "~"
 			(at 25.4 76.2 0)
 			(effects
@@
 			)
 		)
-		(property "Description" ""
+		(property "Description" "Audio Jack, 3 Poles (Stereo / TRS)"
 			(at 25.4 76.2 0)
 			(effects
@@
 			)
 		)
-		(property "Datasheet" "ok : 6"
+		(property "Datasheet" "~"
 			(at 60.96 118.11 0)
 			(effects
@@
 			)
 		)
-		(property "Description" ""
+		(property "Description" "Unpolarized capacitor"
 			(at 60.96 118.11 0)
 			(effects
@@
 			)
 		)
-		(property "Datasheet" "ok 2"
+		(property "Datasheet" "~"
 			(at 25.4 111.76 0)
 			(effects
@@
 			)
 		)
-		(property "Description" ""
+		(property "Description" "Audio Jack, 3 Poles (Stereo / TRS)"
 			(at 25.4 111.76 0)
 			(effects
@@
 			)
 		)
-		(property "Description" ""
+		(property "Description" "Power symbol creates a global label with name \"GND\" , ground"
 			(at 38.1 114.3 0)
 			(effects
@@
 			)
 		)
-		(property "Description" ""
+		(property "Description" "Power symbol creates a global label with name \"+3V3\""
 			(at 116.84 78.74 0)
 			(effects
@@
 			)
 		)
-		(property "Description" ""
+		(property "Description" "Power symbol creates a global label with name \"GND\" , ground"
 			(at 142.24 124.46 0)
 			(effects
@@
 			)
 		)
-		(property "Datasheet" "ok : 6"
+		(property "Datasheet" "~"
 			(at 40.64 120.65 0)
 			(effects
@@
 			)
 		)
-		(property "Description" ""
+		(property "Description" "Resistor"
 			(at 40.64 120.65 0)
 			(effects
@@
 			)
 		)
-		(property "Datasheet" "2 ok"
+		(property "Datasheet" "~"
 			(at 242.57 93.98 0)
 			(effects
@@
 			)
 		)
-		(property "Description" ""
+		(property "Description" "Unpolarized capacitor"
 			(at 242.57 93.98 0)
 			(effects
@@
 			)
 		)
-		(property "Datasheet" "ok : 1"
+		(property "Datasheet" "~"
 			(at 146.05 116.84 0)
 			(effects
@@
 			)
 		)
-		(property "Description" ""
+		(property "Description" "Unpolarized capacitor"
 			(at 146.05 116.84 0)
 			(effects
@@
 			)
 		)
-		(property "Datasheet" "ok: 2"
+		(property "Datasheet" "~"
 			(at 129.54 67.31 0)
 			(effects
@@
 			)
 		)
-		(property "Description" ""
+		(property "Description" "Unpolarized capacitor"
 			(at 129.54 67.31 0)
 			(effects
@@
 			)
 		)
-		(property "Datasheet" "ok : 6"
+		(property "Datasheet" "~"
 			(at 60.96 82.55 0)
 			(effects
@@
 			)
 		)
-		(property "Description" ""
+		(property "Description" "Unpolarized capacitor"
 			(at 60.96 82.55 0)
 			(effects
@@
 			)
 		)
-		(property "Description" ""
+		(property "Description" "Power symbol creates a global label with name \"GND\" , ground"
 			(at 40.64 78.74 0)
 			(effects
@@
 			)
 		)
-		(property "Description" ""
+		(property "Description" "Power symbol creates a global label with name \"GND\" , ground"
 			(at 116.84 88.9 0)
 			(effects
@@
 			)
 		)
-		(property "Datasheet" "dispo 18 k"
+		(property "Datasheet" "~"
 			(at 240.03 149.86 0)
 			(effects
@@
 			)
 		)
-		(property "Description" ""
+		(property "Description" "Resistor"
 			(at 240.03 149.86 0)
 			(effects
@@
 			)
 		)
-		(property "Description" ""
+		(property "Description" "Power symbol creates a global label with name \"GND\" , ground"
 			(at 60.96 78.74 0)
 			(effects
@@
 			)
 		)
-		(property "Datasheet" "1 ok"
+		(property "Datasheet" "~"
 			(at 233.68 87.63 0)
 			(effects
@@
 			)
 		)
-		(property "Description" ""
+		(property "Description" "Two pin crystal"
 			(at 233.68 87.63 0)
 			(effects

Commit message: fix: fix components footprints, resistors, crystal
Parts:
- IC2: footprint SOP65P778X199-28N -> ATM90E26-YU-B:SOP65P778X199-28N
- R1, R2, R3, R4, R9: footprint Resistor_THT:R_Axial_DIN0207_L6.3mm_D2.5mm_P7.62mm_Horizontal -> Resistor_SMD:R_0805_2012Metric_Pad1.20x1.40mm_HandSolder
- Y1: footprint Crystal:Crystal_HC18-U_Vertical -> ABLS:HC_49US-_AT49__1
Changed lines of the file:
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@@
 			)
 		)
-		(property "Footprint" "Resistor_THT:R_Axial_DIN0207_L6.3mm_D2.5mm_P7.62mm_Horizontal"
+		(property "Footprint" "Resistor_SMD:R_0805_2012Metric_Pad1.20x1.40mm_HandSolder"
 			(at 42.418 107.95 90)
 			(effects
@@
 			)
 		)
-		(property "Footprint" "SOP65P778X199-28N"
+		(property "Footprint" "ATM90E26-YU-B:SOP65P778X199-28N"
 			(at 189.23 173.66 0)
 			(effects
@@
 			)
 		)
-		(property "Footprint" "Resistor_THT:R_Axial_DIN0207_L6.3mm_D2.5mm_P7.62mm_Horizontal"
+		(property "Footprint" "Resistor_SMD:R_0805_2012Metric_Pad1.20x1.40mm_HandSolder"
 			(at 42.418 83.82 90)
 			(effects
@@
 			)
 		)
-		(property "Footprint" "Resistor_THT:R_Axial_DIN0207_L6.3mm_D2.5mm_P7.62mm_Horizontal"
+		(property "Footprint" "Resistor_SMD:R_0805_2012Metric_Pad1.20x1.40mm_HandSolder"
 			(at 42.418 72.39 90)
 			(effects
@@
 			)
 		)
-		(property "Footprint" "Resistor_THT:R_Axial_DIN0207_L6.3mm_D2.5mm_P7.62mm_Horizontal"
+		(property "Footprint" "Resistor_SMD:R_0805_2012Metric_Pad1.20x1.40mm_HandSolder"
 			(at 42.418 120.65 90)
 			(effects
@@
 			)
 		)
-		(property "Footprint" "Resistor_THT:R_Axial_DIN0207_L6.3mm_D2.5mm_P7.62mm_Horizontal"
+		(property "Footprint" "Resistor_SMD:R_0805_2012Metric_Pad1.20x1.40mm_HandSolder"
 			(at 240.03 151.638 90)
 			(effects
@@
 			)
 		)
-		(property "Footprint" "Crystal:Crystal_HC18-U_Vertical"
+		(property "Footprint" "ABLS:HC_49US-_AT49__1"
 			(at 233.68 87.63 0)
 			(effects

Commit message: fix: update SMD FP components to handsoldering
Parts:
- C5: footprint Capacitor_SMD:C_0805_2012Metric_Pad1.18x1.45mm_HandSolder -> Capacitor_SMD:C_1210_3225Metric_Pad1.33x2.70mm_HandSolder
Changed lines of the file:
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@@
 			)
 		)
-		(property "Footprint" "Capacitor_SMD:C_0805_2012Metric_Pad1.18x1.45mm_HandSolder"
+		(property "Footprint" "Capacitor_SMD:C_1210_3225Metric_Pad1.33x2.70mm_HandSolder"
 			(at 130.5052 71.12 0)
 			(effects

Commit message: feat: add test points
Parts:
- added TP6: TestPoint, TestPoint:TestPoint_THTPad_D1.5mm_Drill0.7mm, symbol Connector:TestPoint
Connections:
- net GND: now also TP6.1
Changed lines of the file:
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@@
 	)
 	(junction
+		(at 119.38 88.9)
+		(diameter 0)
+		(color 0 0 0 0)
+	)
+	(junction
 		(at 248.92 93.98)
 		(diameter 0)
@@
 	(wire
 		(pts
-			(xy 116.84 88.9) (xy 134.62 88.9)
+			(xy 116.84 88.9) (xy 119.38 88.9)
 		)
 		(stroke
@@
 	(wire
 		(pts
+			(xy 119.38 88.9) (xy 134.62 88.9)
+		)
+		(stroke
+			(width 0)
+			(type default)
+		)
+	)
+	(wire
+		(pts
 			(xy 68.58 96.52) (xy 154.94 96.52)
 		)
@@
 					(unit 1)
 				)
+			)
+		)
+	)
+	(symbol
+		(lib_id "Connector:TestPoint")
+		(at 119.38 88.9 0)
+		(unit 1)
+		(exclude_from_sim no)
+		(in_bom yes)
+		(on_board yes)
+		(dnp no)
+		(fields_autoplaced yes)
+		(property "Reference" "TP6"
+			(at 121.92 84.3279 0)
+			(effects
+				(font
+					(size 1.27 1.27)
+				)
+				(justify left)
+			)
+		)
+		(property "Value" "TestPoint"
+			(at 121.92 86.8679 0)
+			(effects
+				(font
+					(size 1.27 1.27)
+				)
+				(justify left)
+			)
+		)
+		(property "Footprint" "TestPoint:TestPoint_THTPad_D1.5mm_Drill0.7mm"
+			(at 124.46 88.9 0)
+			(effects
+				(font
+					(size 1.27 1.27)
+				)
+				(hide yes)
+			)
+		)
+		(property "Datasheet" "~"
+			(at 124.46 88.9 0)
+			(effects
+				(font
+					(size 1.27 1.27)
+				)
+				(hide yes)
+			)
+		)
+		(property "Description" "test point"
+			(at 119.38 88.9 0)
+			(effects
+				(font
+					(size 1.27 1.27)
+				)
+				(hide yes)
+			)
+		)
+		(pin "1"
+		)
+		(instances
+			(project ""
+				(path "/08ef31dc-81c2-4bcd-8336-e62c344e451e/c04c621c-1838-44d9-9dae-69912433c007"
+					(reference "TP6")
+					(unit 1)
+				)
